Commit message: Update description package

File: ros_ws/src/mw_description/urdf/mw.urdf.xacro (robot description, xacro)
@@ -1,27 +1,130 @@
-<?xml version="1.0" encoding="UTF-8"?>
-<robot xmlns:xacro="http://wiki.ros.org/xacro" name="mw">
-  <!-- Use this if parameters are set from the launch file, otherwise delete -->
-  <xacro:arg name="prefix" default="" />
-  <xacro:arg name="use_mock_hardware" default="false" />
-  <xacro:arg name="mock_sensor_commands" default="false" />
-  <xacro:arg name="sim_gazebo_classic" default="false" />
-  <xacro:arg name="sim_gazebo" default="false" />
-  <xacro:arg name="simulation_controllers" default="" />
-  <xacro:include filename="$(find mw_description)/urdf/mw/mw_macro.xacro"/>
-  <xacro:include filename="$(find mw_description)/urdf/mw/mw_macro.ros2_control.xacro"/>
-  <!-- create link fixed to the "world" -->
-  <link name="world" />
-  <!-- Load robot's macro with parameters -->
-  <!-- set prefix if multiple robots are used -->
-  <xacro:mw prefix="$(arg prefix)" parent="world" >
-    <origin xyz="0 0 0" rpy="0 0 0" />          <!-- position robot in the world -->
-  </xacro:mw>
-  <xacro:mw_ros2_control
-    name="mw"
-    prefix="$(arg prefix)"
-    use_mock_hardware="$(arg use_mock_hardware)"
-    mock_sensor_commands="$(arg mock_sensor_commands)"
-    sim_gazebo_classic="$(arg sim_gazebo_classic)"
-    sim_gazebo="$(arg sim_gazebo)"
-    simulation_controllers="$(arg simulation_controllers)" />
+<?xml version="1.0" encoding="utf-8"?>
+<robot name="mw_car" xmlns:xacro="http://wiki.ros.org/xacro">
+  <xacro:property name="ns" value="mw" />
+  <link name="${ns}/base_footprint" />
+  <!-- common link-->
+  <xacro:macro name="common_link" params="name *origin">
+    <link name="${ns}/${name}">
+      <xacro:insert_block name="origin" />
+    </link>
+  </xacro:macro>
+  <!-- continuous joint-->
+  <xacro:macro name="continuous_joint" params="name parent child xyz rpy axis">
+    <joint name="${ns}/${name}" type="continuous">
+      <parent link="${ns}/${parent}" />
+      <child link="${ns}/${child}" />
+      <origin xyz="${xyz}" rpy="${rpy}" />
+      <axis xyz="${axis}" />
+      <limit lower="${-pi}" upper="${pi}" effort="100" velocity="1" />
+    </joint>
+  </xacro:macro>
+  <!-- fixed joint-->
+  <xacro:macro name="fixed_joint" params="name parent child xyz rpy">
+    <joint name="${ns}/${name}" type="fixed">
+      <parent link="${ns}/${parent}" />
+      <child link="${ns}/${child}" />
+      <origin xyz="${xyz}" rpy="${rpy}" />
+    </joint>
+  </xacro:macro>
+  <link name="${ns}/base_link">
+    <inertial>
+      <origin xyz="-0.0718509386127855 0.00738215784490594 0.119676355791491" rpy="0 0 0" />
+      <mass value="0.486218814966626" />
+      <inertia
+        ixx="0.00196277727666921"
+        ixy="2.50447049446755E-07"
+        ixz="0.000140534767811098"
+        iyy="0.00457256033711368"
+        iyz="2.68618064993882E-07"
+        izz="0.00493927269870476" />
+    </inertial>
+    <visual>
+      <geometry>
+        <mesh filename="package://mw_description/meshes/base_link.STL" />
+      </geometry>
+      <origin xyz="0 0 0" rpy="0 0 0" />
+      <material>
+        <color rgba="0 0.7 0 1" />
+      </material>
+    </visual>
+    <collision>
+      <geometry>
+        <mesh filename="package://mw_description/meshes/base_link.STL" />
+      </geometry>
+      <origin xyz="0 0 0" rpy="0 0 0" />
+    </collision>
+  </link>
+  <xacro:fixed_joint name="base_joint" parent="base_footprint" child="base_link" xyz="0.0 0.0 0.0"
+    rpy="0 0 0" />
+  <xacro:common_link name="front_right_wheel">
+    <inertial>
+      <origin xyz="-0.199063466201963 0.152786006806629 0.0710729630656461" rpy="0 0 0" />
+      <mass value="0.051532" />
+      <inertia ixx="1.4595E-05" ixy="-4.3975E-10" ixz="4.415E-10"
+        iyy="1.4594E-05" iyz="-1.7476E-09" izz="2.4264E-05" />
+    </inertial>
+  </xacro:common_link>
+  <xacro:continuous_joint name="front_right_joint" parent="base_link" child="front_right_wheel"
+    xyz="0.12721 -0.1454 0.048603" rpy="-${pi/2} 0 ${pi}" axis="0 1 0" />
+  <xacro:common_link name="front_left_wheel">
+    <inertial>
+      <origin xyz="-0.199119784807379 -0.138021691116814 0.071103918576079" rpy="0 0 0" />
+      <mass value="0.051543" />
+      <inertia ixx="1.4597E-05" ixy="-4.7945E-10" ixz="-2.4786E-10"
+        iyy="1.4598E-05" iyz="1.7972E-09" izz="2.4267E-05" />
+    </inertial>
+  </xacro:common_link>
+  <xacro:continuous_joint name="front_left_joint" parent="base_link" child="front_left_wheel"
+    xyz="0.12727 0.1454 0.048572" rpy="${pi/2} 0 0" axis="0 1 0" />
+  <xacro:common_link name="back_right_wheel">
+    <inertial>
+      <origin xyz="0.00792558007520176 0.152786006806629 0.0712769954892365" rpy="0 0 0" />
+      <mass value="0.051540174053366" />
+      <inertia ixx="1.45974152250002E-05" ixy="1.94850559178397E-10" ixz="-1.61846387282284E-09"
+        iyy="1.4596501955693E-05" iyz="-6.27904057423818E-10" izz="2.42663091380451E-05" />
+    </inertial>
+  </xacro:common_link>
+  <xacro:continuous_joint name="back_right_joint" parent="base_link" child="back_right_wheel"
+    xyz="-0.079777 -0.1454 0.048399" rpy="-${pi/2} 0 ${pi}" axis="0 1 0" />
+  <xacro:common_link name="back_left_wheel">
+    <inertial>
+      <origin xyz="0.00789687485202048 -0.138021691116814 0.0710896498186508" rpy="0 0 0" />
+      <mass value="0.0515309299357028" />
+      <inertia ixx="1.45942986129926E-05" ixy="-3.19787215398093E-10" ixz="1.74943062058915E-09"
+        iyy="1.45948727598913E-05" iyz="1.61769812110049E-10" izz="2.4263683888153E-05" />
+    </inertial>
+  </xacro:common_link>
+  <xacro:continuous_joint name="back_left_joint" parent="base_link" child="back_left_wheel"
+    xyz="-0.079748 0.1454 0.048587" rpy="${pi/2} 0 0" axis="0 1 0" />
+  <xacro:common_link name="laser_link">
+    <inertial>
+      <origin xyz="-0.205591625169509 0.00738215784490645 -0.0163143442085112" rpy="0 0 0" />
+      <mass value="0.0483909504209895" />
+      <inertia ixx="1.58456966399128E-05" ixy="-4.23913983850005E-07" ixz="-2.09597897904374E-07"
+        iyy="3.89262522903605E-05" iyz="3.24809725932687E-07" izz="4.86230801106223E-05" />
+    </inertial>
+  </xacro:common_link>
+  <xacro:fixed_joint name="laser_joint" parent="base_link" child="laser_link"
+    xyz="0.13374 0 0.13599"
+    rpy="0 0 0" />
+  <xacro:common_link name="camera_link">
+    <inertial>
+      <origin xyz="-0.220993303058215 0.00787952902341162 -0.0803035792325282" rpy="0 0 0" />
+      <mass value="0" />
+      <inertia ixx="0" ixy="0" ixz="0" iyy="0" iyz="0" izz="0" />
+    </inertial>
+  </xacro:common_link>
+  <xacro:fixed_joint name="camera_joint" parent="base_link" child="camera_link"
+    xyz="0.14914 -0.00049737 0.19998" rpy="0 0 0" />
+  <xacro:common_link name="imu_link">
+    <inertial>
+      <origin xyz="-0.216043303058216 -0.0052321578449091 -0.0162763557914886" rpy="0 0 0" />
+      <mass value="0" />
+      <inertia ixx="0" ixy="0" ixz="0"
+        iyy="0" iyz="0" izz="0" />
+    </inertial>
+  </xacro:common_link>
+  <xacro:fixed_joint name="base_imu" parent="base_link" child="imu_link"
+    xyz="0.14419 0.00215 0.1034"
+    rpy="3.1416 0 0" />
 </robot>

Commit message: Update description package

File: ros_ws/src/mw_description/urdf/mw.urdf.xacro (robot description, xacro)
@@ -1,5 +1,5 @@
 <?xml version="1.0" encoding="utf-8"?>
 <robot name="mw_car" xmlns:xacro="http://wiki.ros.org/xacro">
-  <xacro:property name="ns" value="mw" />
+  <xacro:property name="ns" value="" />
   <link name="${ns}/base_footprint" />
   <!-- common link-->

Commit message: Update para

File: ros_ws/src/mw_description/urdf/mw.urdf.xacro (robot description, xacro)
@@ -1,5 +1,5 @@
 <?xml version="1.0" encoding="utf-8"?>
 <robot name="mw_car" xmlns:xacro="http://wiki.ros.org/xacro">
-  <xacro:property name="ns" value="" />
+  <xacro:property name="ns" value="mw" />
   <link name="${ns}/base_footprint" />
   <!-- common link-->
